File: merch-board/audio.kicad_sch (KiCad schematic)
At the start: 18 parts, among them U4 PCM5100A, U5 TPA6211A1DGN

Commit message: Add LCSC part numbers
Parts:
- C17, C21, C24: value 0.1u -> 100n; LCSC C14663 -> C1525
- C18, C19, C22: LCSC C19702 -> C15525
- C20: LCSC C23630 -> C12530
- C25: LCSC C1604 -> C1531
- C29: LCSC C15849 -> C14445
- R10, R9: footprint Resistor_SMD:R_0402_1005Metric -> Resistor_SMD:R_0603_1608Metric
- R7: LCSC C209149 -> C25117
Changed lines of the file:
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@@
 			)
 		)
-		(property "Value" "0.1u"
+		(property "Value" "100n"
 			(at 138.811 120.404 0)
 			(effects
@@
 			)
 		)
-		(property "LCSC" "C14663"
+		(property "LCSC" "C1525"
 			(at 135.89 119.38 0)
 			(effects
@@
 			)
 		)
-		(property "LCSC" "C15849"
+		(property "LCSC" "C14445"
 			(at 257.81 77.47 0)
 			(effects
@@
 			)
 		)
-		(property "Footprint" "Resistor_SMD:R_0402_1005Metric"
+		(property "Footprint" "Resistor_SMD:R_0603_1608Metric"
 			(at 200.66 99.568 90)
 			(effects
@@
 			)
 		)
-		(property "LCSC" "C209149"
+		(property "LCSC" "C25117"
 			(at 123.19 91.44 0)
 			(effects
@@
 			)
 		)
-		(property "Footprint" "Resistor_SMD:R_0402_1005Metric"
+		(property "Footprint" "Resistor_SMD:R_0603_1608Metric"
 			(at 200.66 102.108 90)
 			(effects
@@
 			)
 		)
-		(property "LCSC" "C1604"
+		(property "LCSC" "C1531"
 			(at 143.51 102.87 0)
 			(effects
@@
 			)
 		)
-		(property "LCSC" "C19702"
+		(property "LCSC" "C15525"
 			(at 72.39 76.2 0)
 			(effects
@@
 			)
 		)
-		(property "Value" "0.1u"
+		(property "Value" "100n"
 			(at 117.221 120.404 0)
 			(effects
@@
 			)
 		)
-		(property "LCSC" "C14663"
+		(property "LCSC" "C1525"
 			(at 114.3 119.38 0)
 			(effects
@@
 			)
 		)
-		(property "LCSC" "C23630"
+		(property "LCSC" "C12530"
 			(at 107.95 104.14 0)
 			(effects
@@
 			)
 		)
-		(property "LCSC" "C19702"
+		(property "LCSC" "C15525"
 			(at 104.14 119.38 0)
 			(effects
@@
 			)
 		)
-		(property "LCSC" "C19702"
+		(property "LCSC" "C15525"
 			(at 125.73 119.38 0)
 			(effects
@@
 			)
 		)
-		(property "Value" "0.1u"
+		(property "Value" "100n"
 			(at 65.151 77.224 0)
 			(effects
@@
 			)
 		)
-		(property "LCSC" "C14663"
+		(property "LCSC" "C1525"
 			(at 62.23 76.2 0)
 			(effects

Commit message: Update BOM
Parts:
- C26, C27, C28: LCSC C21120 -> C16772
Changed lines of the file:
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@@
 			)
 		)
-		(property "LCSC" "C21120"
+		(property "LCSC" "C16772"
 			(at 238.76 113.03 0)
 			(effects
@@
 			)
 		)
-		(property "LCSC" "C21120"
+		(property "LCSC" "C16772"
 			(at 190.5 106.68 0)
 			(effects
@@
 			)
 		)
-		(property "LCSC" "C21120"
+		(property "LCSC" "C16772"
 			(at 189.23 97.79 0)
 			(effects
